File: arduino.sch (KiCad schematic (older format))
At the start: 0 parts

Commit message: Module 3 Unit 9
Understanding The Arduino Module
Parts:
- added ARD?: ARDUINO, symbol ARDUINO
- added R? (x13): R, ~, symbol R
Connections:
- net MISO: now also R?.2
- net MOSI: now also R?.2
- net Relay+: now also R?.2
- net Relay-: now also R?.2
- net SCLK: now also R?.2
- net TACH_MEAS: now also R?.1
- new net: ARD?.11 (D0_RX), R?.1
- new net: ARD?.12 (D1_TX), R?.1
- new net: ARD?.19 (D8), R?.1
- new net: ARD?.20 (D9_PWM0), R?.1
- new net: ARD?.21 (CS), R?.1
- new net: ARD?.22 (MOSI), R?.1
- new net: ARD?.23 (MISO), R?.1
- new net: ARD?.24 (SCK), R?.1
- new net: ARD?.5 (A0), R?.2
- new net: ARD?.6 (A1), R?.2
- new net: ARD?.7 (A2), R?.2
- new net: ARD?.8 (A3), R?.2
- new net ADC_CS_N: R?.2
- new net Current_Measure: R?.1
- new net DAC_CS_N: R?.2
- new net Fan_En_N: R?.2
- new net GND: R?.1
- new net LED_EN_PWM: R?.2
- new net V+ADJ_MON: R?.1
- new net V-ADJ_MON: R?.1

Commit message: Module 3 Unit 10
Revisiting The Current/Fan Module
Parts:
- added R? (x2): R, ~, symbol R
Connections:
- net at ARD?.11 (D0_RX): now also R?.1; no longer R?.1
- net at ARD?.18 (D7): now also R?.1
- net at ARD?.21 (CS): now also R?.1; no longer R?.1
- net at ARD?.4 (9V): now also R?.2
- net Fan_En_N renamed FAN_PWM
- new net +12P: R?.1
- new net FAN_MODE: R?.2
Other:
- moved on the sheet: R?
Changed lines of the file:
@@
 Text HLabel 6500 3300 2    60   Output ~ 0
 SCLK
+Text HLabel 6500 3900 2    60   Output ~ 0
+DAC_CS_N
 Text HLabel 6500 3600 2    60   Output ~ 0
-DAC_CS_N
-Text HLabel 6500 4600 2    60   Output ~ 0
-Fan_En_N
+FAN_PWM
 Text HLabel 3300 4400 0    60   Input ~ 0
 TACH_MEAS
@@
 L R R?
 U 1 1 5300AF8A
-P 6050 4600
-F 0 "R?" V 6130 4600 40  0000 C CNN
-F 1 "R" V 6057 4601 40  0000 C CNN
-F 2 "~" V 5980 4600 30  0000 C CNN
-F 3 "~" H 6050 4600 30  0000 C CNN
-	1    6050 4600
-	0    -1   -1   0
-$EndComp
-Wire Wire Line
-	5800 4600 5600 4600
-Wire Wire Line
-	6500 4600 6300 4600
+P 6050 3600
+F 0 "R?" V 6130 3600 40  0000 C CNN
+F 1 "R" V 6057 3601 40  0000 C CNN
+F 2 "~" V 5980 3600 30  0000 C CNN
+F 3 "~" H 6050 3600 30  0000 C CNN
+	1    6050 3600
+	0    -1   -1   0
+$EndComp
+Wire Wire Line
+	5800 3600 5600 3600
+Wire Wire Line
+	6500 3600 6300 3600
 $Comp
 L R R?
@@
 L R R?
 U 1 1 5300CD6A
-P 6050 3600
-F 0 "R?" V 6130 3600 40  0000 C CNN
-F 1 "R" V 6057 3601 40  0000 C CNN
-F 2 "~" V 5980 3600 30  0000 C CNN
-F 3 "~" H 6050 3600 30  0000 C CNN
-	1    6050 3600
+P 6050 3900
+F 0 "R?" V 6130 3900 40  0000 C CNN
+F 1 "R" V 6057 3901 40  0000 C CNN
+F 2 "~" V 5980 3900 30  0000 C CNN
+F 3 "~" H 6050 3900 30  0000 C CNN
+	1    6050 3900
 	0    -1   -1   0
 $EndComp
@@
 	6300 3500 6500 3500
 Wire Wire Line
-	6300 3600 6500 3600
+	6300 3900 6500 3900
 Wire Wire Line
 	5600 3300 5800 3300
@@
 	5600 3500 5800 3500
 Wire Wire Line
-	5600 3600 5800 3600
+	5600 3900 5800 3900
 $Comp
 L R R?
@@
 Wire Wire Line
 	6500 3800 6300 3800
+Text HLabel 6500 4600 2    60   Input ~ 0
+FAN_MODE
+$Comp
+L R R?
+U 1 1 530106D9
+P 6050 4600
+F 0 "R?" V 6130 4600 40  0000 C CNN
+F 1 "R" V 6057 4601 40  0000 C CNN
+F 2 "~" V 5980 4600 30  0000 C CNN
+F 3 "~" H 6050 4600 30  0000 C CNN
+	1    6050 4600
+	0    -1   -1   0
+$EndComp
+Wire Wire Line
+	5600 4600 5800 4600
+Wire Wire Line
+	6300 4600 6500 4600
+$Comp
+L R R?
+U 1 1 5301106A
+P 3750 3950
+F 0 "R?" V 3830 3950 40  0000 C CNN
+F 1 "R" V 3757 3951 40  0000 C CNN
+F 2 "~" V 3680 3950 30  0000 C CNN
+F 3 "~" H 3750 3950 30  0000 C CNN
+	1    3750 3950
+	0    -1   -1   0
+$EndComp
+Wire Wire Line
+	4200 3950 4000 3950
+$Comp
+L +12P #PWR?
+U 1 1 53011090
+P 3250 3850
+F 0 "#PWR?" H 3250 3820 30  0001 C CNN
+F 1 "+12P" H 3250 3950 30  0000 C CNN
+F 2 "" H 3250 3850 60  0000 C CNN
+F 3 "" H 3250 3850 60  0000 C CNN
+	1    3250 3850
+	1    0    0    -1
+$EndComp
+Wire Wire Line
+	3500 3950 3250 3950
+Wire Wire Line
+	3250 3950 3250 3850
 $EndSCHEMATC
