File: power.sch (KiCad schematic (older format))
At the start: 0 parts

Commit message: Module 3 Unit 6
Understanding The Power Protection And Filtering Module
Parts:
- added C? (x2): C, ~, symbol C
- added F? (x4): FUSE, ~, symbol FUSE
- added L? (x2): INDUCTOR, ~, symbol INDUCTOR
- added P?: CONN_12X2, symbol CONN_12X2
- added R?: R, ~, symbol R
- added SW?: SWITCH_INV, ~, symbol SWITCH_INV
Connections:
- net labels added: +12P, +12V, +3.3V, +5V, -12P, -12V, GND
- wire segments 0 -> 38

Commit message: Module 3 Unit 10
Revisiting The Current/Fan Module
Parts:
- removed F? (x4): FUSE, ~, symbol FUSE
- added TH? (x4): THERMISTOR, ~, symbol THERMISTOR
Connections:
- net labels added: +12C
- wire segments 38 -> 39
Changed lines of the file:
@@
 $Descr A4 11693 8268
 encoding utf-8
-Sheet 5 9
+Sheet 4 9
 Title ""
 Date "16 feb 2014"
@@
 	1    0    0    -1
 $EndComp
-$Comp
-L FUSE F?
-U 1 1 52F953F7
-P 2700 1200
-F 0 "F?" H 2800 1250 40  0000 C CNN
-F 1 "FUSE" H 2600 1150 40  0000 C CNN
-F 2 "~" H 2700 1200 60  0000 C CNN
-F 3 "~" H 2700 1200 60  0000 C CNN
-	1    2700 1200
-	1    0    0    -1
-$EndComp
-$Comp
-L FUSE F?
-U 1 1 52F95404
-P 3200 1300
-F 0 "F?" H 3300 1350 40  0000 C CNN
-F 1 "FUSE" H 3100 1250 40  0000 C CNN
-F 2 "~" H 3200 1300 60  0000 C CNN
-F 3 "~" H 3200 1300 60  0000 C CNN
-	1    3200 1300
-	1    0    0    -1
-$EndComp
-$Comp
-L FUSE F?
-U 1 1 52F9540A
-P 3700 1600
-F 0 "F?" H 3800 1650 40  0000 C CNN
-F 1 "FUSE" H 3600 1550 40  0000 C CNN
-F 2 "~" H 3700 1600 60  0000 C CNN
-F 3 "~" H 3700 1600 60  0000 C CNN
-	1    3700 1600
-	1    0    0    -1
-$EndComp
-$Comp
-L FUSE F?
-U 1 1 52F95410
-P 4200 1800
-F 0 "F?" H 4300 1850 40  0000 C CNN
-F 1 "FUSE" H 4100 1750 40  0000 C CNN
-F 2 "~" H 4200 1800 60  0000 C CNN
-F 3 "~" H 4200 1800 60  0000 C CNN
-	1    4200 1800
-	1    0    0    -1
-$EndComp
 Wire Wire Line
 	1400 1300 800  1300
@@
 	8700 2700 8700 2950
 Connection ~ 7750 2700
+$Comp
+L +12C #PWR?
+U 1 1 5300EC5D
+P 2350 700
+F 0 "#PWR?" H 2350 670 30  0001 C CNN
+F 1 "+12C" H 2350 810 40  0000 C CNN
+F 2 "" H 2350 700 60  0000 C CNN
+F 3 "" H 2350 700 60  0000 C CNN
+	1    2350 700
+	1    0    0    -1
+$EndComp
+Wire Wire Line
+	2350 1600 2350 700
+Connection ~ 2350 1600
+$Comp
+L THERMISTOR TH?
+U 1 1 5300F414
+P 4200 1800
+F 0 "TH?" V 4300 1850 50  0000 C CNN
+F 1 "THERMISTOR" V 4100 1800 50  0000 C CNN
+F 2 "~" H 4200 1800 60  0000 C CNN
+F 3 "~" H 4200 1800 60  0000 C CNN
+	1    4200 1800
+	0    -1   -1   0
+$EndComp
+$Comp
+L THERMISTOR TH?
+U 1 1 5300F421
+P 2700 1200
+F 0 "TH?" V 2800 1250 50  0000 C CNN
+F 1 "THERMISTOR" V 2600 1200 50  0000 C CNN
+F 2 "~" H 2700 1200 60  0000 C CNN
+F 3 "~" H 2700 1200 60  0000 C CNN
+	1    2700 1200
+	0    -1   -1   0
+$EndComp
+$Comp
+L THERMISTOR TH?
+U 1 1 5300F427
+P 3200 1300
+F 0 "TH?" V 3300 1350 50  0000 C CNN
+F 1 "THERMISTOR" V 3100 1300 50  0000 C CNN
+F 2 "~" H 3200 1300 60  0000 C CNN
+F 3 "~" H 3200 1300 60  0000 C CNN
+	1    3200 1300
+	0    -1   -1   0
+$EndComp
+$Comp
+L THERMISTOR TH?
+U 1 1 5300F42D
+P 3700 1600
+F 0 "TH?" V 3800 1650 50  0000 C CNN
+F 1 "THERMISTOR" V 3600 1600 50  0000 C CNN
+F 2 "~" H 3700 1600 60  0000 C CNN
+F 3 "~" H 3700 1600 60  0000 C CNN
+	1    3700 1600
+	0    -1   -1   0
+$EndComp
 $EndSCHEMATC
