File: led driver.sch (KiCad schematic (older format))
At the start: 0 parts

Commit message: Module 3 Unit 8
Understanding The LED Driver Module
Parts:
- added C? (x2): C, ~, symbol C
- added D?: ZENER, ~, symbol ZENER
- added L?: INDUCTOR, ~, symbol INDUCTOR
- added R?: R, ~, symbol R
- added U?: AP5726, symbol AP5726
Connections:
- net String+: now also C?.1, D?.2 (K), U?.5 (OVP)
- net String-: now also R?.1, U?.3 (FB)
- new net: D?.1 (A), L?.2, U?.1 (SW)
- new net +5V: C?.1, L?.1, U?.6 (VIN)
- new net GND: C?.2, C?.2, R?.2, U?.2 (GND)
- new net LED_EN_PWM: U?.4 (EN)
Changed lines of the file:
@@
 Comment4 ""
 $EndDescr
-Text HLabel 1700 1800 0    60   Input ~ 0
-EN
-Text HLabel 1700 2000 0    60   Input ~ 0
-FREQ
-Text HLabel 9450 1800 2    60   Output ~ 0
+Text HLabel 1650 2900 0    60   Input ~ 0
+LED_EN_PWM
+Text HLabel 8200 1700 2    60   Output ~ 0
 String+
-Text HLabel 9450 2050 2    60   Input ~ 0
+Text HLabel 8200 2900 2    60   Input ~ 0
 String-
+$Comp
+L AP5726 U?
+U 1 1 52FFEA34
+P 3000 2800
+F 0 "U?" H 2650 2350 60  0000 C CNN
+F 1 "AP5726" H 3000 2750 60  0000 C CNN
+F 2 "" H 3000 2950 60  0000 C CNN
+F 3 "" H 3000 2950 60  0000 C CNN
+	1    3000 2800
+	1    0    0    -1
+$EndComp
+Wire Wire Line
+	1650 2900 2300 2900
+$Comp
+L +5V #PWR?
+U 1 1 52FFF652
+P 2200 1400
+F 0 "#PWR?" H 2200 1490 20  0001 C CNN
+F 1 "+5V" H 2200 1490 30  0000 C CNN
+F 2 "" H 2200 1400 60  0000 C CNN
+F 3 "" H 2200 1400 60  0000 C CNN
+	1    2200 1400
+	1    0    0    -1
+$EndComp
+$Comp
+L GND #PWR?
+U 1 1 52FFF661
+P 3100 3850
+F 0 "#PWR?" H 3100 3850 30  0001 C CNN
+F 1 "GND" H 3100 3780 30  0001 C CNN
+F 2 "" H 3100 3850 60  0000 C CNN
+F 3 "" H 3100 3850 60  0000 C CNN
+	1    3100 3850
+	1    0    0    -1
+$EndComp
+$Comp
+L GND #PWR?
+U 1 1 52FFF66E
+P 2200 2600
+F 0 "#PWR?" H 2200 2600 30  0001 C CNN
+F 1 "GND" H 2200 2530 30  0001 C CNN
+F 2 "" H 2200 2600 60  0000 C CNN
+F 3 "" H 2200 2600 60  0000 C CNN
+	1    2200 2600
+	1    0    0    -1
+$EndComp
+$Comp
+L C C?
+U 1 1 52FFF680
+P 2200 2200
+F 0 "C?" H 2200 2300 40  0000 L CNN
+F 1 "C" H 2206 2115 40  0000 L CNN
+F 2 "~" H 2238 2050 30  0000 C CNN
+F 3 "~" H 2200 2200 60  0000 C CNN
+	1    2200 2200
+	1    0    0    -1
+$EndComp
+$Comp
+L ZENER D?
+U 1 1 52FFF6B9
+P 4100 1700
+F 0 "D?" H 4100 1800 50  0000 C CNN
+F 1 "ZENER" H 4100 1600 40  0000 C CNN
+F 2 "~" H 4100 1700 60  0000 C CNN
+F 3 "~" H 4100 1700 60  0000 C CNN
+	1    4100 1700
+	1    0    0    -1
+$EndComp
+$Comp
+L R R?
+U 1 1 52FFF6D2
+P 4900 3350
+F 0 "R?" V 4980 3350 40  0000 C CNN
+F 1 "R" V 4907 3351 40  0000 C CNN
+F 2 "~" V 4830 3350 30  0000 C CNN
+F 3 "~" H 4900 3350 30  0000 C CNN
+	1    4900 3350
+	1    0    0    -1
+$EndComp
+$Comp
+L C C?
+U 1 1 52FFF6DF
+P 7000 2000
+F 0 "C?" H 7000 2100 40  0000 L CNN
+F 1 "C" H 7006 1915 40  0000 L CNN
+F 2 "~" H 7038 1850 30  0000 C CNN
+F 3 "~" H 7000 2000 60  0000 C CNN
+	1    7000 2000
+	1    0    0    -1
+$EndComp
+Wire Wire Line
+	2200 2600 2200 2400
+Wire Wire Line
+	2200 2000 2200 1400
+Wire Wire Line
+	3100 3850 3100 3450
+Wire Wire Line
+	3700 2750 4450 2750
+Wire Wire Line
+	4450 2750 4450 1700
+Connection ~ 4450 1700
+Wire Wire Line
+	7000 1800 7000 1700
+Wire Wire Line
+	4300 1700 8200 1700
+Connection ~ 7000 1700
+Wire Wire Line
+	3100 3700 4900 3700
+Wire Wire Line
+	4900 3700 4900 3600
+Connection ~ 3100 3700
+Wire Wire Line
+	4900 3100 4900 2900
+Wire Wire Line
+	3700 2900 8200 2900
+Connection ~ 4900 2900
+$Comp
+L GND #PWR?
+U 1 1 52FFF8FA
+P 7000 2500
+F 0 "#PWR?" H 7000 2500 30  0001 C CNN
+F 1 "GND" H 7000 2430 30  0001 C CNN
+F 2 "" H 7000 2500 60  0000 C CNN
+F 3 "" H 7000 2500 60  0000 C CNN
+	1    7000 2500
+	1    0    0    -1
+$EndComp
+Wire Wire Line
+	7000 2500 7000 2200
+$Comp
+L INDUCTOR L?
+U 1 1 52FFF937
+P 3200 1700
+F 0 "L?" V 3150 1700 40  0000 C CNN
+F 1 "INDUCTOR" V 3300 1700 40  0000 C CNN
+F 2 "~" H 3200 1700 60  0000 C CNN
+F 3 "~" H 3200 1700 60  0000 C CNN
+	1    3200 1700
+	0    -1   -1   0
+$EndComp
+Wire Wire Line
+	2900 1700 2200 1700
+Connection ~ 2200 1700
+Wire Wire Line
+	3500 1700 3900 1700
+Wire Wire Line
+	3250 2200 3250 2000
+Wire Wire Line
+	3250 2000 3700 2000
+Wire Wire Line
+	3700 2000 3700 1700
+Connection ~ 3700 1700
+Wire Wire Line
+	2950 2200 2950 2000
+Wire Wire Line
+	2950 2000 2700 2000
+Wire Wire Line
+	2700 2000 2700 1700
+Connection ~ 2700 1700
 $EndSCHEMATC

Commit message: Module 3 Unit 9
Understanding The Arduino Module
Connections:
- net String+ renamed LED_String+
- net String- renamed LED_String-
Changed lines of the file:
@@
 Sheet 6 9
 Title ""
-Date "15 feb 2014"
+Date "16 feb 2014"
 Rev ""
 Comp ""
@@
 LED_EN_PWM
 Text HLabel 8200 1700 2    60   Output ~ 0
-String+
-Text HLabel 8200 2900 2    60   Input ~ 0
-String-
+LED_String+
+Text HLabel 8200 2900 2    60   Output ~ 0
+LED_String-
 $Comp
 L AP5726 U?
