File: relay.sch (KiCad schematic (older format))
At the start: 0 parts

Commit message: Module 3 Unit 5
Understanding The Relay Module
Parts:
- added D?: LED, ~, symbol LED
- added D?: DIODE, ~, symbol DIODE
- added K?: RELAY_SPDT, ~, symbol RELAY_SPDT
- added Q?: NPN, ~, symbol NPN
- added R? (x6): R, ~, symbol R
- added U?: PHTRANS, ~, symbol PHTRANS
Connections:
- net DIN+: now also U?.1
- net DIN-: now also R?.1
- new net: R?.2, U?.2
- new net: D?.1 (A), R?.1, U?.4
- new net: D?.2 (K), K?.2 (COIL+), R?.1, R?.2, U?.5
- new net: R?.1, U?.6
- new net: Q?.2 (B), R?.2
- new net: Q?.1 (E), R?.2
- new net: D?.1 (A), K?.5 (COIL-), Q?.3 (C)
- new net: D?.2 (K), R?.2
- new net +12P: R?.2
- new net COM: K?.1 (COM)
- new net GND: R?.1, R?.1
- new net NC: K?.4 (NC)
- new net NO: K?.3 (NO)
Changed lines of the file:
@@
 LIBS:contrib
 LIBS:valves
+LIBS:benchbudee
 LIBS:benchbudee-cache
 EELAYER 27 0
@@
 Comment4 ""
 $EndDescr
-Text HLabel 1650 2050 0    60   Input ~ 0
+Text HLabel 1600 3600 0    60   Input ~ 0
 DIN+
-Text HLabel 1650 2250 0    60   Output ~ 0
+Text HLabel 1600 3950 0    60   Output ~ 0
 DIN-
-Text HLabel 9250 1950 2    60   Input ~ 0
-Relay+
-Text HLabel 9250 2250 2    60   Output ~ 0
-Relay-
+Text HLabel 9250 2700 2    60   BiDi ~ 0
+NC
+Text HLabel 9250 2900 2    60   BiDi ~ 0
+NO
+$Comp
+L PHTRANS U?
+U 1 1 52F930D8
+P 3200 3800
+F 0 "U?" H 3150 4150 70  0000 C CNN
+F 1 "PHTRANS" H 3150 3450 70  0000 C CNN
+F 2 "~" H 3200 3800 60  0000 C CNN
+F 3 "~" H 3200 3800 60  0000 C CNN
+	1    3200 3800
+	1    0    0    -1
+$EndComp
+$Comp
+L R R?
+U 1 1 52F930F6
+P 4650 4000
+F 0 "R?" V 4730 4000 40  0000 C CNN
+F 1 "R" V 4657 4001 40  0000 C CNN
+F 2 "~" V 4580 4000 30  0000 C CNN
+F 3 "~" H 4650 4000 30  0000 C CNN
+	1    4650 4000
+	0    -1   -1   0
+$EndComp
+$Comp
+L NPN Q?
+U 1 1 52F93105
+P 6600 4000
+F 0 "Q?" H 6600 3850 50  0000 R CNN
+F 1 "NPN" H 6600 4150 50  0000 R CNN
+F 2 "~" H 6600 4000 60  0000 C CNN
+F 3 "~" H 6600 4000 60  0000 C CNN
+	1    6600 4000
+	1    0    0    -1
+$EndComp
+$Comp
+L LED D?
+U 1 1 52F93114
+P 4100 4500
+F 0 "D?" H 4100 4600 50  0000 C CNN
+F 1 "LED" H 4100 4400 50  0000 C CNN
+F 2 "~" H 4100 4500 60  0000 C CNN
+F 3 "~" H 4100 4500 60  0000 C CNN
+	1    4100 4500
+	0    1    1    0
+$EndComp
+$Comp
+L RELAY_SPDT K?
+U 1 1 52F936F2
+P 7350 2850
+F 0 "K?" H 7600 2450 70  0000 C CNN
+F 1 "RELAY_SPDT" H 7350 3200 70  0000 C CNN
+F 2 "~" H 7350 2950 60  0000 C CNN
+F 3 "~" H 7350 2950 60  0000 C CNN
+	1    7350 2850
+	1    0    0    -1
+$EndComp
+Text HLabel 9250 2000 2    60   BiDi ~ 0
+COM
+$Comp
+L R R?
+U 1 1 52F9374C
+P 6700 5150
+F 0 "R?" V 6780 5150 40  0000 C CNN
+F 1 "R" V 6707 5151 40  0000 C CNN
+F 2 "~" V 6630 5150 30  0000 C CNN
+F 3 "~" H 6700 5150 30  0000 C CNN
+	1    6700 5150
+	-1   0    0    1
+$EndComp
+$Comp
+L GND #PWR?
+U 1 1 52F9376B
+P 6700 5850
+F 0 "#PWR?" H 6700 5850 30  0001 C CNN
+F 1 "GND" H 6700 5780 30  0001 C CNN
+F 2 "" H 6700 5850 60  0000 C CNN
+F 3 "" H 6700 5850 60  0000 C CNN
+	1    6700 5850
+	1    0    0    -1
+$EndComp
+$Comp
+L R R?
+U 1 1 52F9378B
+P 4100 5150
+F 0 "R?" V 4180 5150 40  0000 C CNN
+F 1 "R" V 4107 5151 40  0000 C CNN
+F 2 "~" V 4030 5150 30  0000 C CNN
+F 3 "~" H 4100 5150 30  0000 C CNN
+	1    4100 5150
+	-1   0    0    1
+$EndComp
+$Comp
+L R R?
+U 1 1 52F938EE
+P 4400 2650
+F 0 "R?" V 4480 2650 40  0000 C CNN
+F 1 "R" V 4407 2651 40  0000 C CNN
+F 2 "~" V 4330 2650 30  0000 C CNN
+F 3 "~" H 4400 2650 30  0000 C CNN
+	1    4400 2650
+	-1   0    0    1
+$EndComp
+$Comp
+L +12P #PWR?
+U 1 1 52F938F6
+P 4400 2000
+F 0 "#PWR?" H 4400 1970 30  0001 C CNN
+F 1 "+12P" H 4400 2100 30  0000 C CNN
+F 2 "" H 4400 2000 60  0000 C CNN
+F 3 "" H 4400 2000 60  0000 C CNN
+	1    4400 2000
+	1    0    0    -1
+$EndComp
+$Comp
+L R R?
+U 1 1 52F93939
+P 4100 3600
+F 0 "R?" V 4180 3600 40  0000 C CNN
+F 1 "R" V 4107 3601 40  0000 C CNN
+F 2 "~" V 4030 3600 30  0000 C CNN
+F 3 "~" H 4100 3600 30  0000 C CNN
+	1    4100 3600
+	0    -1   -1   0
+$EndComp
+$Comp
+L R R?
+U 1 1 52F93A9C
+P 2150 3950
+F 0 "R?" V 2230 3950 40  0000 C CNN
+F 1 "R" V 2157 3951 40  0000 C CNN
+F 2 "~" V 2080 3950 30  0000 C CNN
+F 3 "~" H 2150 3950 30  0000 C CNN
+	1    2150 3950
+	0    -1   -1   0
+$EndComp
+$Comp
+L DIODE D?
+U 1 1 52F93B5A
+P 5800 3300
+F 0 "D?" H 5800 3400 40  0000 C CNN
+F 1 "DIODE" H 5800 3200 40  0000 C CNN
+F 2 "~" H 5800 3300 60  0000 C CNN
+F 3 "~" H 5800 3300 60  0000 C CNN
+	1    5800 3300
+	0    -1   -1   0
+$EndComp
+Wire Wire Line
+	7750 2700 9250 2700
+Wire Wire Line
+	9250 2900 7750 2900
+Wire Wire Line
+	3750 4000 4400 4000
+Wire Wire Line
+	4900 4000 6400 4000
+Wire Wire Line
+	6700 4900 6700 4200
+Wire Wire Line
+	6700 5400 6700 5850
+Wire Wire Line
+	4100 4000 4100 4300
+Connection ~ 4100 4000
+Wire Wire Line
+	4100 4700 4100 4900
+Wire Wire Line
+	4100 5400 4100 5600
+Wire Wire Line
+	4100 5600 6700 5600
+Connection ~ 6700 5600
+Wire Wire Line
+	4400 2400 4400 2000
+Wire Wire Line
+	4400 2900 4400 3800
+Wire Wire Line
+	4400 3800 3750 3800
+Wire Wire Line
+	3750 3600 3850 3600
+Wire Wire Line
+	4350 3600 4400 3600
+Connection ~ 4400 3600
+Wire Wire Line
+	2650 3600 1600 3600
+Wire Wire Line
+	1600 3950 1900 3950
+Wire Wire Line
+	2400 3950 2650 3950
+Wire Wire Line
+	6950 2800 6700 2800
+Wire Wire Line
+	6700 2800 6700 2000
+Wire Wire Line
+	6700 2000 9250 2000
+Wire Wire Line
+	6950 3100 6700 3100
+Wire Wire Line
+	6700 3100 6700 3800
+Wire Wire Line
+	6950 3000 4400 3000
+Connection ~ 4400 3000
+Wire Wire Line
+	5800 3100 5800 3000
+Connection ~ 5800 3000
+Wire Wire Line
+	5800 3500 5800 3600
+Wire Wire Line
+	5800 3600 6700 3600
+Connection ~ 6700 3600
 $EndSCHEMATC

Commit message: Module 3 Unit 9
Understanding The Arduino Module
Connections:
- net COM renamed RELAY_COM
- net DIN+ renamed Relay+
- net DIN- renamed Relay-
- net NC renamed RELAY_NC
- net NO renamed RELAY_NO
Changed lines of the file:
@@
 $Descr A4 11693 8268
 encoding utf-8
-Sheet 4 9
+Sheet 3 9
 Title ""
-Date "15 feb 2014"
+Date "16 feb 2014"
 Rev ""
 Comp ""
@@
 $EndDescr
 Text HLabel 1600 3600 0    60   Input ~ 0
-DIN+
+Relay+
 Text HLabel 1600 3950 0    60   Output ~ 0
-DIN-
+Relay-
 Text HLabel 9250 2700 2    60   BiDi ~ 0
-NC
+RELAY_NC
 Text HLabel 9250 2900 2    60   BiDi ~ 0
-NO
+RELAY_NO
 $Comp
 L PHTRANS U?
@@
 $EndComp
 Text HLabel 9250 2000 2    60   BiDi ~ 0
-COM
+RELAY_COM
 $Comp
 L R R?
