File: thermocouple.sch (KiCad schematic (older format))
At the start: 0 parts

Commit message: Module 2 Unit 14
Defining Your Inputs and Outputs
Changed lines of the file:
@@
 LIBS:contrib
 LIBS:valves
-LIBS:benchbudee-block-cache
+LIBS:benchbudee-cache
 EELAYER 27 0
 EELAYER END
@@
 Sheet 3 8
 Title ""
-Date "1 feb 2014"
+Date "2 feb 2014"
 Rev ""
 Comp ""
@@
 Text HLabel 9650 3100 2    60   Input ~ 0
 tc in -
+Text HLabel 2700 2400 0    60   Input ~ 0
+MOSI
+Text HLabel 2700 2600 0    60   Output ~ 0
+MISO
+Text HLabel 2700 2800 0    60   Input ~ 0
+SCLK
+Text HLabel 2700 3000 0    60   Input ~ 0
+CS_N
 $EndSCHEMATC

Commit message: Module 3 Unit 3
Understanding the Thermocouple Module
Parts:
- added D?: ZENER, ~, symbol ZENER
- added R? (x7): R, ~, symbol R
- added U? (x4): LM324, symbol LM324
- added U? (x2): MCP3550-60-E/SN, SO8, symbol MCP3550-60-E/SN
Connections:
- net CS_N: now also U?.7 (~CS~)
- net MISO: now also U?.6 (SDO/~RDY~)
- net SCLK: now also U?.5 (SCK)
- net tc in +: now also U?.3 (+)
- net tc in -: now also U?.3 (+)
- new net: R?.1, R?.2, U?.1
- new net: R?.1, R?.2, U?.2 (-) (x3)
- new net: R?.2, R?.2, U?.1
- new net: R?.1, U?.1, U?.2 (Vin+)
- new net: R?.1, R?.2, U?.3 (+)
- new net: U?.1, U?.2 (-), U?.2 (Vin+)
- new net +12V: D?.2 (K), U?.3 (+), U?.4 (V+), U?.4 (V+), U?.4 (V+)
- new net -12V: U?.11 (V-), U?.11 (V-), U?.11 (V-)
- new net AGND: D?.1 (A), R?.1, U?.3 (Vin-), U?.3 (Vin-)
Other:
- note added: "16-24 bit ADC"
- note added: "Analog/TC Input"
- note added: "General Temperature Sensor"
- note added: "Instrumentation Amplifier"

Commit message: Module 3 Unit 9
Understanding The Arduino Module
Connections:
- net tc in + renamed TC_IN+
- net tc in - renamed TC_IN-
Changed lines of the file:
@@
 Sheet 3 9
 Title ""
-Date "15 feb 2014"
+Date "16 feb 2014"
 Rev ""
 Comp ""
@@
 $EndDescr
 Text HLabel 10550 1800 2    60   Input ~ 0
-tc in +
+TC_IN+
 Text HLabel 10500 4800 2    60   Input ~ 0
-tc in -
+TC_IN-
 Text HLabel 2700 2400 0    60   Input ~ 0
 MOSI
